File: ParaMETEO-reset-adapter.kicad_pcb (KiCad board)
At the start: 2 copper layers, 40.4 x 20.8 mm, 18 parts, among them J1 1WIRE, J2 Screw_Terminal_01x06, U1 FODM217A, U2 FODM217A, U3 MCP130T-300I/TT, U4 LTV-824, X1 SHF-105-01-L-D-SM

Commit message: final version pushed do jblpcb
Parts:
- removed BT1: Battery_Cell, battery_keystone:BAT_1074
- removed U4: LTV-824, Package_DIP:DIP-8_W7.62mm
- added J3: BAT-, Connector_Wire:SolderWire-1.5sqmm_1x01_D1.7mm_OD3.9mm, F.Cu at (173.0, 61.9)
- added J4: BAT+, Connector_Wire:SolderWire-1.5sqmm_1x01_D1.7mm_OD3.9mm, F.Cu at (138.7, 61.9)
- added R10: 0, Resistor_SMD:R_0805_2012Metric_Pad1.20x1.40mm_HandSolder, F.Cu at (155.1, 57.2)
- added R8: 1k, Resistor_SMD:R_0805_2012Metric_Pad1.20x1.40mm_HandSolder, F.Cu at (155.1, 54.0)
- added R9: 0, Resistor_SMD:R_0805_2012Metric_Pad1.20x1.40mm_HandSolder, F.Cu at (140.8, 67.8)
- moved R2 84.0 mm to (165.9, 62.9)
- moved R3 79.7 mm to (161.8, 64.0)
- moved R4 76.4 mm to (159.2, 59.1)
- moved R5 67.4 mm to (150.2, 59.0)
- moved C1 64.5 mm to (149.7, 63.6), turned to 180 degrees
- moved R1 60.9 mm to (138.9, 71.0)
- moved R6 44.2 mm to (138.4, 56.4), turned to -90 degrees
- moved U2 41.6 mm to (171.8, 69.8), turned to 0 degrees
- moved R7 40.7 mm to (141.4, 57.0)
- moved U3 10.1 mm to (153.6, 62.9)
- moved J2 9.79 mm to (147.8, 52.7)
- moved U1 4.19 mm to (167.9, 65.9)
- moved J1 0.11 mm to (171.3, 53.6)
Connections:
- J1 pad 3: GNDD -> unconnected-(J1-Pin_3-Pad3)
- J1 pad 4: (no net) -> unconnected-(J1-Pin_4-Pad4)
- J1 pad 5: (no net) -> GNDD
- J1 pad 6: (no net) -> GNDD
- R4 pad 1: BAT_BOOT -> /B+
- R5 pad 1: BAT_BOOT -> /B+
- X1 pad 7: unconnected-(X1-Pad7) -> BOOT_CONN
Routing:
- net GNDD: track 0.00 -> 81.5 mm, vias 0 -> 4
- net RESET: track 0.00 -> 61.9 mm, vias 0 -> 2
- net GND: track 0.00 -> 50.4 mm, vias 0 -> 2
- net Net-(R9-Pad1): track 0.00 -> 37.6 mm, vias 0 -> 2
- net /B+: track 0.00 -> 35.5 mm, vias 0 -> 2
- net TO_RESET_IN: track 0.00 -> 31.9 mm, vias 0 -> 2
- net Net-(R1-Pad2): track 0.00 -> 30.1 mm, vias 0 -> 1
- net BAT_BOOT: track 0.00 -> 29.0 mm, vias 0 -> 2
- net TO_BOOT_IN: track 0.00 -> 26.3 mm, vias 0 -> 1
- net +3.3V: track 0.00 -> 24.0 mm
- net FOR_BOOT_OUT: track 0.00 -> 20.1 mm, vias 0 -> 1
- net FOR_RESET_OUT: track 0.00 -> 12.9 mm
- net BOOT_CONN: track 0.00 -> 10.3 mm
- net Net-(R2-Pad2): track 0.00 -> 7.05 mm
- net Net-(J2-Pin_5): track 0.00 -> 6.43 mm
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Other:
- board size 40.4 x 20.8 mm -> 40.4 x 21.5 mm
- board text added: "BOOT"
- board text added: "BOOT CON"
- board text added: "BOOT-3.3"
- board text added: "BOOT-B+"
- board text added: "GND"
- board text added: "GNDD"
- board text added: "RESET"
- board text added: "RST"
