File: ParaMETEO-reset-adapter.kicad_sch (KiCad schematic)
At the start: 18 parts, among them J1 1WIRE, J2 Screw_Terminal_01x06, U1 FODM217A, U2 FODM217A, U3 MCP130T-300I/TT, U4 LTV-824, X1 SHF-105-01-L-D-SM

Commit message: final version pushed do jblpcb
Parts:
- removed BT1: Battery_Cell, battery_keystone:BAT_1074, symbol bat_keystone:1074
- removed U4: LTV-824, Package_DIP:DIP-8_W7.62mm, symbol Isolator:LTV-824
- added J3: BAT-, Connector_Wire:SolderWire-1.5sqmm_1x01_D1.7mm_OD3.9mm, symbol Connector:Screw_Terminal_01x01
- added J4: BAT+, Connector_Wire:SolderWire-1.5sqmm_1x01_D1.7mm_OD3.9mm, symbol Connector:Screw_Terminal_01x01
- added R10, R9: 0, Resistor_SMD:R_0805_2012Metric_Pad1.20x1.40mm_HandSolder, symbol Device:R
- added R8: 1k, Resistor_SMD:R_0805_2012Metric_Pad1.20x1.40mm_HandSolder, symbol Device:R
- J1: symbol Connector:Screw_Terminal_01x03 -> Connector:Screw_Terminal_01x06
Connections:
- net +3.3V: now also R10.1
- net BAT_BOOT: now also R10.2, R8.2; no longer R4.1, R5.1
- net GND: now also J3.1 (Pin_1)
- net GNDD: now also J1.5 (Pin_5), J1.6 (Pin_6); no longer J1.3 (Pin_3)
- net at TP2.1, U1.3: now also R9.1
- net BOOT_CONN: now reaches X1.7
- net BOOT_CONN: now also R9.2
- new net B+: J4.1 (Pin_1), R4.1, R5.1, R8.1
Other:
- moved on the sheet: C1, R2, R5, U2, U3
